Commit message: started with tests

File: master_thesis_ros/catkin_ws/src/turtlebot3_vlp16_description/urdf/VLP-16.urdf.xacro (robot description, xacro)
@@ -10,9 +10,9 @@
     <link name="${name}_base_link">
       <inertial>
-        <mass value="0.1"/>
+        <mass value="0.01"/>
         <origin xyz="0 0 0.03585"/>
-        <inertia ixx="${(0.1 * (3.0*0.0516*0.0516 + 0.0717*0.0717)) / 12.0}" ixy="0" ixz="0"
-          iyy="${(0.1 * (3.0*0.0516*0.0516 + 0.0717*0.0717)) / 12.0}" iyz="0"
-          izz="${0.5 * 0.1 * (0.0516*0.0516)}"/>
+        <inertia ixx="${(0.01 * (3.0*0.0516*0.0516 + 0.0717*0.0717)) / 12.0}" ixy="0" ixz="0"
+          iyy="${(0.01 * (3.0*0.0516*0.0516 + 0.0717*0.0717)) / 12.0}" iyz="0"
+          izz="${0.5 * 0.01 * (0.0516*0.0516)}"/>
       </inertial>
       <visual>

File: master_thesis_ros/catkin_ws/src/turtlebot3_vlp16_description/urdf/turtlebot3_waffle.urdf.xacro (robot description, xacro)
@@ -140,5 +140,5 @@
    <!-- Velodyne -->
   <xacro:VLP-16 parent="base_link" name="velodyne" topic="/velodyne_points" hz="10" samples="440" gpu="true" max_range="30.0">
-    <origin xyz="-0.15 0 0.1" rpy="0 0 0"/>
+    <origin xyz="-0.15 0 0.35" rpy="0 0 0"/>
   </xacro:VLP-16>
 </robot>
